File: code/project/drone/electronics/main.brd (EAGLE design)
At the start: 100 x 80 mm, 80 parts, among them IC1 CD74HCT4067M, T1 BTIRF3710S, T16 BTIRF3710S, T17 BTIRF3710S, T18 BTIRF3710S, T19 BTIRF3710S, T2 BTIRF3710S, T20 BTIRF3710S, T21 BTIRF3710S, T22 BTIRF3710S, T23 BTIRF3710S, T24 BTIRF3710S, T3 BTIRF3710S, U1 74HC595N, U2 ESP8266-NODEMCU, U3 74HC595N

Commit message: update
Parts:
- added J5: Batterie_IN, 0IUT CONNECTEURS:MSTBA2
- added PS1: TSR_1-2450E, TSR_1-2450E:TSR12450E
- added PS2: TSR_1-2433E, TSR_1-2433E:TSR-1-2433
Connections:
- removed net VCC: C1.2, C2.1, C3.1, IC1.24, J1.2, J2.2, J3.2, J4.2, R1.2, R11.2, R16.2, R24.2, R25.2, R6.2, U1.10, U1.16, U3.10, U3.16
- removed net VIN: U2.15
- new net +24V: J1.2, J2.2, J3.2, J4.2, J5.1, PS1.1, PS2.1, R1.2, R11.2, R16.2, R6.2
- new net +5V: PS1.3, U2.15
- net +3,3V: now also C1.2, C2.1, C3.1, IC1.24, PS2.3, R24.2, R25.2, U1.10, U1.16, U3.10, U3.16
- net GND: now also J5.2, PS1.2, PS2.2

Commit message: udpate
Connections:
- net N$15: now also IC1.7; no longer IC1.8
- net N$23: now also IC1.8, R17.2; no longer IC1.7, R12.2
- net N$31: now also IC1.9, R12.2; no longer IC1.6, R17.2
- net N$7: now also IC1.6; no longer IC1.9
Changed lines of the file:
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@@
 <wire x1="24.13" y1="59.69" x2="38.1762" y2="74.93" width="0" layer="19" extent="1-1"/>
-</signal>
-<signal name="N$7">
-<contactref element="R2" pad="2"/>
-<contactref element="IC1" pad="9"/>
-<wire x1="-104.8766" y1="130.81" x2="-148.235" y2="-18.415" width="0" layer="19" extent="1-1"/>
 </signal>
 <signal name="N$9">
@@
 <wire x1="52.07" y1="59.69" x2="55.9562" y2="74.93" width="0" layer="19" extent="1-1"/>
 </signal>
-<signal name="N$15">
-<contactref element="R7" pad="2"/>
-<contactref element="IC1" pad="8"/>
-<wire x1="-40.1066" y1="138.43" x2="-148.235" y2="-17.145" width="0" layer="19" extent="1-1"/>
-</signal>
 <signal name="N$16">
 <contactref element="R10" pad="2"/>
@@
 <wire x1="-35.56" y1="78.74" x2="73.7362" y2="74.93" width="0" layer="19" extent="1-1"/>
 </signal>
-<signal name="N$23">
-<contactref element="R12" pad="2"/>
-<contactref element="IC1" pad="7"/>
-<wire x1="-71.8566" y1="138.43" x2="-148.235" y2="-15.875" width="0" layer="19" extent="1-1"/>
-</signal>
 <signal name="N$24">
 <contactref element="R15" pad="2"/>
@@
 <wire x1="-77.47" y1="78.74" x2="-95.25" y2="132.08" width="0" layer="19" extent="1-1"/>
 <wire x1="20.3962" y1="74.93" x2="-18.3134" y2="144.78" width="0" layer="19" extent="1-1"/>
-</signal>
-<signal name="N$31">
-<contactref element="R17" pad="2"/>
-<contactref element="IC1" pad="6"/>
-<wire x1="-103.6066" y1="138.43" x2="-148.235" y2="-14.605" width="0" layer="19" extent="1-1"/>
 </signal>
 <signal name="N$32">
@@
 <wire x1="-162.56" y1="-203.2" x2="-161.29" y2="-193.04" width="0" layer="19" extent="1-1"/>
 </signal>
+<signal name="N$7">
+<contactref element="IC1" pad="6"/>
+<contactref element="R2" pad="2"/>
+<wire x1="-104.8766" y1="130.81" x2="-148.235" y2="-14.605" width="0" layer="19" extent="1-1"/>
+</signal>
+<signal name="N$15">
+<contactref element="R7" pad="2"/>
+<contactref element="IC1" pad="7"/>
+<wire x1="-40.1066" y1="138.43" x2="-148.235" y2="-15.875" width="0" layer="19" extent="1-1"/>
+</signal>
+<signal name="N$23">
+<contactref element="R17" pad="2"/>
+<contactref element="IC1" pad="8"/>
+<wire x1="-103.6066" y1="138.43" x2="-148.235" y2="-17.145" width="0" layer="19" extent="1-1"/>
+</signal>
+<signal name="N$31">
+<contactref element="IC1" pad="9"/>
+<contactref element="R12" pad="2"/>
+<wire x1="-71.8566" y1="138.43" x2="-148.235" y2="-18.415" width="0" layer="19" extent="1-1"/>
+</signal>
 </signals>
