File: code/project/drone/electronics/main.sch (EAGLE design)
At the start: 61 parts, among them T10 TRANSISTOR_DRONE, T11 TRANSISTOR_DRONE, T12 TRANSISTOR_DRONE, T13 TRANSISTOR_DRONE, T14 TRANSISTOR_DRONE, T15 TRANSISTOR_DRONE, T4 TRANSISTOR_DRONE, T5 TRANSISTOR_DRONE, T6 TRANSISTOR_DRONE, T7 TRANSISTOR_DRONE, T8 TRANSISTOR_DRONE, T9 TRANSISTOR_DRONE, U1 ESP32-EV1.0

Commit message: add files
Parts:
- removed T10, T11, T12, T13, T14, T15, T4, T5, T6, T7, T8, T9: TRANSISTOR_DRONE, composant_sa_mere(avec_l'intentonation):TRANSISTOR_DRONE
- added T1, T16, T17, T18, T19, T2, T20, T21, T22, T23, T24, T3: BTIRF3710S, librairie_drone:BTIRF3710S
Connections:
- net GND: now also T1.S, T16.S, T17.S, T18.S, T19.S, T2.S, T20.S, T21.S, T22.S, T23.S, T24.S, T3.S; no longer T10.E, T11.E, T12.E, T13.E, T14.E, T15.E, T4.E, T5.E, T6.E, T7.E, T8.E, T9.E
- net N$1: now also T2.D; no longer T5.C
- net N$10: now also T17.G; no longer T8.B
- net N$12: now also T18.G; no longer T9.B
- net N$13: now also T17.D; no longer T8.C
- net N$14: now also T16.D; no longer T7.C
- net N$16: now also T18.D; no longer T9.C
- net N$17: now also T19.G; no longer T10.B
- net N$18: now also T20.G; no longer T11.B
- net N$20: now also T21.G; no longer T12.B
- net N$21: now also T20.D; no longer T11.C
- net N$22: now also T19.D; no longer T10.C
- net N$24: now also T21.D; no longer T12.C
- net N$25: now also T22.G; no longer T13.B
- net N$26: now also T23.G; no longer T14.B
- net N$28: now also T24.G; no longer T15.B
- net N$29: now also T23.D; no longer T14.C
- net N$3: now also T1.G; no longer T4.B
- net N$30: now also T22.D; no longer T13.C
- net N$32: now also T24.D; no longer T15.C
- net N$4: now also T2.G; no longer T5.B
- net N$5: now also T3.G; no longer T6.B
- net N$6: now also T1.D; no longer T4.C
- net N$8: now also T16.G; no longer T7.B
- net N$9: now also T3.D; no longer T6.C
Other:
- moved on the sheet: D1, D10, D11, D12, D13, D14, D15, D16, D17, D18, D19, D2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

Commit message: end of electric card
Parts:
- added C1: 0.1u, 0IUT RLCQ:C-CMS1206
- added C2, C3: 100n, 0IUT RLCQ:C-CMS1206
- added IC1: CD74HCT4067M, CD74HCT4067M:CD74HCT4067M
- added JP1: sdCard, jumper:JP4E
- added JP2: analog_cam, jumper:JP4E
- added JP3: digital_cam, jumper:JP4E
- added JP4: digital_cam_2, jumper:JP4E
- added JP5: sd_alim, jumper:JP1E
- added JP6: (no value), jumper:JP1E
- added JP7: cam_alim, jumper:JP1E
- added JP8: cam_rst_pwdn, jumper:JP1E
- added R21, R24, R25: 10k, 0IUT RLCQ:R-CMS1206
- added R22, R23: 4.7k, 0IUT RLCQ:R-CMS1206
- added U2: ESP8266-NODEMCU, 0IUT xPROJETS:ESP8266-NODEMCU
- added U3: 74HC595N, 0IUT CI LOGIQUES:74HC595N
- U1: value ESP32-EV1.0 -> 74HC595N; device 0IUT xPROJETS:ESP32-EV1.0 -> 0IUT CI LOGIQUES:74HC595N
Connections:
- new net +3,3V: JP5.1, JP7.1, JP8.1, U2.3V3
- new net N$33: JP1.1, U1G$1.Q0
- new net N$34: JP1.2, U1G$1.Q1
- new net N$35: JP1.3, U1G$1.Q2
- new net N$36: JP1.4, U1G$1.Q3
- new net N$37: IC1.S3, U3G$1.Q1
- new net N$38: C1.1, IC1.GND
- new net N$39: IC1.S2, U3G$1.Q0
- new net N$40: IC1.S1, U3G$1.Q2
- new net N$41: IC1.S0, U3G$1.Q3
- new net N$42: IC1.COMMON_INPUT/OUTPUT, U2.A0
- new net N$43: IC1.!E, R21.2
- new net N$44: U1G$1.SHCP, U2.D0
- new net N$45: U1G$1.STCP, U2.D1
- new net N$46: U1G$1.DS, U2.D2
- new net N$47: JP3.1, U1G$1.Q4
- new net N$48: JP3.2, U1G$1.Q5
- new net N$49: JP3.3, U1G$1.Q6
- new net N$50: JP3.4, U1G$1.Q7
- new net N$51: IC1.I4, JP2.4
- new net N$52: IC1.I5, JP2.3
- new net N$53: IC1.I6, JP2.2
- new net N$54: IC1.I7, JP2.1
- new net N$55: U2.D3, U3G$1.SHCP
- new net N$56: U2.D4, U3G$1.STCP
- new net N$57: U2.D5, U3G$1.DS
- new net N$58: JP4.1, U3G$1.Q4
- new net N$59: JP4.2, U3G$1.Q5
- new net N$60: JP4.3, U3G$1.Q6
- new net N$61: JP4.4, R22.2
- new net N$62: IC1.I15, JP6.1, R25.1
- new net N$63: R22.1, R23.2, U3G$1.Q7
- new net N$64: IC1.I14, JP6.2, R24.1
- net GND: now also C2.2, C3.2, JP5.2, JP7.2, JP8.2, R21.1, R23.1, U1G$1.!OE!, U1P.GND, U2.GND, U3G$1.!OE!, U3P.GND
- net N$15: now also IC1.I1; no longer U1.A1/39
- net N$23: now also IC1.I2; no longer U1.A2/34
- net N$31: now also IC1.I3; no longer U1.A3/35
- net N$7: now also IC1.I0; no longer U1.A0/36
- net VCC: now also C1.2, C2.1, C3.1, IC1.VCC, R24.2, R25.2, U1G$1.!MR!, U1P.VCC, U3G$1.!MR!, U3P.VCC
Other:
- moved on the sheet: J1, J2

Commit message: update
Parts:
- added J5: Batterie_IN, 0IUT CONNECTEURS:BORNIER_2-D2P
- added PS1: TSR_1-2450E, TSR_1-2450E:TSR_1-2450E
- added PS2: TSR_1-2433E, TSR_1-2433E:TSR_1-2433E
Connections:
- removed net VCC: C1.2, C2.1, C3.1, IC1.VCC, J1.2, J2.2, J3.2, J4.2, R1.2, R11.2, R16.2, R24.2, R25.2, R6.2, U1G$1.!MR!, U1P.VCC, U3G$1.!MR!, U3P.VCC
- new net +24V: J1.2, J2.2, J3.2, J4.2, J5.1, PS1.+VIN, PS2.VIN+, R1.2, R11.2, R16.2, R6.2
- new net +5V: PS1.+VOUT, U2.VIN
- net +3,3V: now also C1.2, C2.1, C3.1, IC1.VCC, PS2.VOUT+, R24.2, R25.2, U1G$1.!MR!, U1P.VCC, U3G$1.!MR!, U3P.VCC
- net GND: now also J5.2, PS1.GND, PS2.GND

Commit message: udpate
Connections:
- net N$15: now also IC1.I2; no longer IC1.I1
- net N$23: now also IC1.I1, R17.2; no longer IC1.I2, R12.2
- net N$31: now also IC1.I0, R12.2; no longer IC1.I3, R17.2
- net N$7: now also IC1.I3; no longer IC1.I0
Other:
- moved on the sheet: C1, C2, C3, D1, D10, D11, D12, D13, D14, D15, D16, D17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
